Commit message: 增加dh_stand_shoulder

File: resources/robots/x1/urdf/x1.urdf (robot description, URDF)
Before this commit: robot x1, 58 links, 57 joints
Joints:
- joint left_shoulder_pitch_joint: limit lower=-3.14 upper=3.14 effort=0 velocity=0 -> lower=-1.2 upper=1.2 effort=40 velocity=6; type fixed -> revolute
- joint right_shoulder_pitch_joint: limit lower=-3.14 upper=3.14 effort=0 velocity=0 -> lower=-1.2 upper=1.2 effort=40 velocity=6; type fixed -> revolute
